File: Schematic/gateLights/power.sch (KiCad schematic (older format))
At the start: 10 parts, among them U7 MC33063A

Commit message: Add inputs
Parts:
- L1: footprint Inductors:Inductor_Taiyo-Yuden_MD-5050 -> GateLight:SCD1005
Changed lines of the file:
@@
 $Descr A4 11693 8268
 encoding utf-8
-Sheet 4 5
+Sheet 4 6
 Title "Power Supplies"
 Date "2017-05-20"
@@
 $EndComp
 $Comp
-L GND #PWR12
+L GND #PWR010
 U 1 1 592069BC
 P 3900 4600
-F 0 "#PWR12" H 3900 4350 50  0001 C CNN
+F 0 "#PWR010" H 3900 4350 50  0001 C CNN
 F 1 "GND" H 3900 4450 50  0000 C CNN
 F 2 "" H 3900 4600 50  0001 C CNN
@@
 $EndComp
 $Comp
-L GND #PWR13
+L GND #PWR011
 U 1 1 59206A8E
 P 4850 4600
-F 0 "#PWR13" H 4850 4350 50  0001 C CNN
+F 0 "#PWR011" H 4850 4350 50  0001 C CNN
 F 1 "GND" H 4850 4450 50  0000 C CNN
 F 2 "" H 4850 4600 50  0001 C CNN
@@
 F 0 "L1" V 5100 3550 50  0000 C CNN
 F 1 "100uH" V 5225 3550 50  0000 C CNN
-F 2 "Inductors:Inductor_Taiyo-Yuden_MD-5050" H 5150 3550 50  0001 C CNN
+F 2 "GateLight:SCD1005" H 5150 3550 50  0001 C CNN
 F 3 "" H 5150 3550 50  0001 C CNN
 F 4 "SCD1005T-101K-N 100U/1A YAGEO" V 5150 3550 60  0001 C CNN "VALUE"
@@
 $EndComp
 $Comp
-L GND #PWR14
+L GND #PWR012
 U 1 1 59206E85
 P 5350 4650
-F 0 "#PWR14" H 5350 4400 50  0001 C CNN
+F 0 "#PWR012" H 5350 4400 50  0001 C CNN
 F 1 "GND" H 5350 4500 50  0000 C CNN
 F 2 "" H 5350 4650 50  0001 C CNN
@@
 	5350 3550 5350 3750
 $Comp
-L GND #PWR15
+L GND #PWR013
 U 1 1 59206F5B
 P 5700 4650
-F 0 "#PWR15" H 5700 4400 50  0001 C CNN
+F 0 "#PWR013" H 5700 4400 50  0001 C CNN
 F 1 "GND" H 5700 4500 50  0000 C CNN
 F 2 "" H 5700 4650 50  0001 C CNN
@@
 $EndComp
 $Comp
-L GND #PWR17
+L GND #PWR014
 U 1 1 59206F7E
 P 6150 4650
-F 0 "#PWR17" H 6150 4400 50  0001 C CNN
+F 0 "#PWR014" H 6150 4400 50  0001 C CNN
 F 1 "GND" H 6150 4500 50  0000 C CNN
 F 2 "" H 6150 4650 50  0001 C CNN
@@
 $EndComp
 $Comp
-L GND #PWR11
+L GND #PWR015
 U 1 1 5920710A
 P 3250 4600
-F 0 "#PWR11" H 3250 4350 50  0001 C CNN
+F 0 "#PWR015" H 3250 4350 50  0001 C CNN
 F 1 "GND" H 3250 4450 50  0000 C CNN
 F 2 "" H 3250 4600 50  0001 C CNN
@@
 	3250 3750 3500 3750
 $Comp
-L +5V #PWR16
+L +5V #PWR016
 U 1 1 592071DA
 P 6150 3200
-F 0 "#PWR16" H 6150 3050 50  0001 C CNN
+F 0 "#PWR016" H 6150 3050 50  0001 C CNN
 F 1 "+5V" H 6150 3340 50  0000 C CNN
 F 2 "" H 6150 3200 50  0001 C CNN
@@
 Connection ~ 6150 3550
 $Comp
-L GND #PWR9
+L GND #PWR017
 U 1 1 5920723D
 P 2450 4600
-F 0 "#PWR9" H 2450 4350 50  0001 C CNN
+F 0 "#PWR017" H 2450 4350 50  0001 C CNN
 F 1 "GND" H 2450 4450 50  0000 C CNN
 F 2 "" H 2450 4600 50  0001 C CNN
@@
 $EndComp
 $Comp
-L GND #PWR10
+L GND #PWR018
 U 1 1 59207319
 P 2800 4600
-F 0 "#PWR10" H 2800 4350 50  0001 C CNN
+F 0 "#PWR018" H 2800 4350 50  0001 C CNN
 F 1 "GND" H 2800 4450 50  0000 C CNN
 F 2 "" H 2800 4600 50  0001 C CNN
