File: Schematic/gateLights/input.sch (KiCad schematic (older format))
At the start: 12 parts, among them Q1 2N7002, Q2 2N7002, Q3 2N7002

Commit message: Fix resistor footprints
Parts:
- R10, R11, R12, R13, R16, R17: footprint Resistors_SMD:R_1210_HandSoldering -> Resistors_SMD:R_1206_HandSoldering
- R14, R15, R18: footprint Resistors_SMD:R_1210_HandSoldering -> Resistors_SMD:R_0603_HandSoldering
Changed lines of the file:
@@
 F 0 "R10" V 3330 3100 50  0000 C CNN
 F 1 "27K" V 3250 3100 50  0000 C CNN
-F 2 "Resistors_SMD:R_1210_HandSoldering" V 3180 3100 50  0001 C CNN
+F 2 "Resistors_SMD:R_1206_HandSoldering" V 3180 3100 50  0001 C CNN
 F 3 "" H 3250 3100 50  0001 C CNN
 	1    3250 3100
@@
 F 0 "R11" V 3330 3550 50  0000 C CNN
 F 1 "10K" V 3250 3550 50  0000 C CNN
-F 2 "Resistors_SMD:R_1210_HandSoldering" V 3180 3550 50  0001 C CNN
+F 2 "Resistors_SMD:R_1206_HandSoldering" V 3180 3550 50  0001 C CNN
 F 3 "" H 3250 3550 50  0001 C CNN
 	1    3250 3550
@@
 F 0 "R14" V 4230 2750 50  0000 C CNN
 F 1 "10K" V 4150 2750 50  0000 C CNN
-F 2 "Resistors_SMD:R_1210_HandSoldering" V 4080 2750 50  0001 C CNN
+F 2 "Resistors_SMD:R_0603_HandSoldering" V 4080 2750 50  0001 C CNN
 F 3 "" H 4150 2750 50  0001 C CNN
 	1    4150 2750
@@
 F 0 "R12" V 3330 5550 50  0000 C CNN
 F 1 "27K" V 3250 5550 50  0000 C CNN
-F 2 "Resistors_SMD:R_1210_HandSoldering" V 3180 5550 50  0001 C CNN
+F 2 "Resistors_SMD:R_1206_HandSoldering" V 3180 5550 50  0001 C CNN
 F 3 "" H 3250 5550 50  0001 C CNN
 	1    3250 5550
@@
 F 0 "R13" V 3330 6000 50  0000 C CNN
 F 1 "10K" V 3250 6000 50  0000 C CNN
-F 2 "Resistors_SMD:R_1210_HandSoldering" V 3180 6000 50  0001 C CNN
+F 2 "Resistors_SMD:R_1206_HandSoldering" V 3180 6000 50  0001 C CNN
 F 3 "" H 3250 6000 50  0001 C CNN
 	1    3250 6000
@@
 F 0 "R15" V 4230 5200 50  0000 C CNN
 F 1 "10K" V 4150 5200 50  0000 C CNN
-F 2 "Resistors_SMD:R_1210_HandSoldering" V 4080 5200 50  0001 C CNN
+F 2 "Resistors_SMD:R_0603_HandSoldering" V 4080 5200 50  0001 C CNN
 F 3 "" H 4150 5200 50  0001 C CNN
 	1    4150 5200
@@
 F 0 "R16" V 7480 3250 50  0000 C CNN
 F 1 "27K" V 7400 3250 50  0000 C CNN
-F 2 "Resistors_SMD:R_1210_HandSoldering" V 7330 3250 50  0001 C CNN
+F 2 "Resistors_SMD:R_1206_HandSoldering" V 7330 3250 50  0001 C CNN
 F 3 "" H 7400 3250 50  0001 C CNN
 	1    7400 3250
@@
 F 0 "R17" V 7480 3700 50  0000 C CNN
 F 1 "10K" V 7400 3700 50  0000 C CNN
-F 2 "Resistors_SMD:R_1210_HandSoldering" V 7330 3700 50  0001 C CNN
+F 2 "Resistors_SMD:R_1206_HandSoldering" V 7330 3700 50  0001 C CNN
 F 3 "" H 7400 3700 50  0001 C CNN
 	1    7400 3700
@@
 F 0 "R18" V 8380 2900 50  0000 C CNN
 F 1 "10K" V 8300 2900 50  0000 C CNN
-F 2 "Resistors_SMD:R_1210_HandSoldering" V 8230 2900 50  0001 C CNN
+F 2 "Resistors_SMD:R_0603_HandSoldering" V 8230 2900 50  0001 C CNN
 F 3 "" H 8300 2900 50  0001 C CNN
 	1    8300 2900
